Commit message: URDF and visualization fixups

File: ur5/ur5.urdf (robot description, URDF)
Before this commit: robot ur5_robotiq85, 22 links, 21 joints
Links:
- link base_link: geometry collision mesh filename=meshes/ur5/collision/base.stl; visual mesh filename=meshes/ur5/visual/base.dae
- link forearm_link: geometry collision mesh filename=meshes/ur5/collision/forearm.stl; visual mesh filename=meshes/ur5/visual/forearm.dae
- link fts_robotside: geometry collision mesh filename=meshes/robotiq_fts300.stl; visual mesh filename=meshes/robotiq_fts300.stl
- link robotiq_85_base_link: geometry collision mesh filename=meshes/robotiq/robotiq_85_base_link_fine.STL; visual mesh filename=meshes/robotiq/robotiq_85_base_link_fine.STL
- link shoulder_link: geometry collision mesh filename=meshes/ur5/collision/shoulder.stl; visual mesh filename=meshes/ur5/visual/shoulder.dae
- link upper_arm_link: geometry collision mesh filename=meshes/ur5/collision/upperarm.stl; visual mesh filename=meshes/ur5/visual/upperarm.dae
- link wrist_1_link: geometry collision mesh filename=meshes/ur5/collision/wrist1.stl; visual mesh filename=meshes/ur5/visual/wrist1.dae
- link wrist_2_link: geometry collision mesh filename=meshes/ur5/collision/wrist2.stl; visual mesh filename=meshes/ur5/visual/wrist2.dae
- link wrist_3_link: geometry collision mesh filename=meshes/ur5/collision/wrist3.stl; visual mesh filename=meshes/ur5/visual/wrist3.dae
